File: pcb/muxi/eagle/muxi.brd (EAGLE design)
At the start: 22.8 x 49.2 mm, 21 parts

Commit message: merge with v05 branch
Parts:
- JP1: device SparkFun-Connectors:1X08_PIN1_NO_SILK -> SparkFun-Connectors:1X06_NO_SILK
- moved JP1 5.35 mm to (7.87, 39.6)
- moved 1 1.18 mm to (3.50, 26.1)
- moved 5 1.18 mm to (3.50, 13.4)
- moved 7 1.18 mm to (3.50, 7.04)
- moved 8 1.18 mm to (3.50, 3.87)
- moved 2 1.18 mm to (3.50, 22.9)
- moved 3 1.18 mm to (3.50, 19.7)
- moved 4 1.18 mm to (3.50, 16.6)
- moved 6 1.18 mm to (3.50, 10.2)
- moved C1 0.86 mm to (11.7, 45.2)
- moved U$2 0.47 mm to (18.7, 4.09)
- moved R1 0.44 mm to (17.4, 27.2)
- moved R2 0.44 mm to (17.4, 24.7)
- moved R3 0.44 mm to (17.4, 22.1)
- moved R5 0.44 mm to (17.4, 17.0)
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Connections:
- removed net DGND: 4051.6, 4051.7, 4051.8, C1.2, JP1.2
- removed net VDD_3V3: 4051.16, C1.1, JP1.1
- net A: now also JP1.4; no longer JP1.5
- net AOUT: now also JP1.2; no longer JP1.8
- net B: now also JP1.5; no longer JP1.6
- net C: now also JP1.6; no longer JP1.7
- net GNDA_ADC: now also 4051.6, 4051.7, 4051.8, C1.2, JP1.3; no longer JP1.4
- net VDD_ADC: now also 4051.16, C1.1, JP1.1; no longer JP1.3
Routing:
- net GNDA_ADC: track 0.00 -> 78.4 mm
- net DGND: track 48.1 -> 0.00 mm
- net AOUT: track 27.4 -> 11.2 mm, vias 2 -> 0
- net VDD_3V3: track 12.6 -> 0.00 mm
- net AIN2: track 38.6 -> 27.1 mm, vias 1 -> 0
- net AIN7: track 41.3 -> 31.3 mm
- net AIN3: track 34.8 -> 27.4 mm
- net VDD_ADC: track 41.1 -> 48.1 mm
- net AIN1: track 29.6 -> 23.7 mm, vias 1 -> 0
- net AIN6: track 39.8 -> 34.1 mm
- net AIN5: track 30.4 -> 25.6 mm
- net AIN0: track 22.5 -> 18.2 mm
- net AIN4: track 31.5 -> 27.6 mm
- net C: track 3.59 -> 2.50 mm
- net A: track 3.59 -> 2.55 mm
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Other:
- board text added: "3.3V"
- board text added: "A"
- board text added: "B"
- board text added: "C"
- board text added: "CC BY-SA 3.0"
- board text added: "Designed by: I. Franco,"
- board text added: "H. Venkatesan and A. Tom"
- board text added: "IDMIL"
- board text added: "PRYNTH MUXI V0.5"
- board text removed: "IDMIL 2016"
- board text removed: "Ivan Franco"
- board text removed: "Muxi 0.3"
- board text removed: "VDD"
