File: pcb/muxi/eagle/muxi.sch (EAGLE design)
At the start: 19 parts

Commit message: merge with v05 branch
Parts:
- JP1: device SparkFun-Connectors:M08 -> SparkFun-Connectors:M06NO_SILK
Connections:
- removed net DGND: 4051.INH, 4051.VEE, 4051.VSS, C1.-, JP1.2
- removed net VDD_3V3: 4051.VDD, C1.+, JP1.1
- net A: now also JP1.4; no longer JP1.5
- net AOUT: now also JP1.2; no longer JP1.8
- net B: now also JP1.5; no longer JP1.6
- net C: now also JP1.6; no longer JP1.7
- net GNDA_ADC: now also 4051.INH, 4051.VEE, 4051.VSS, C1.-, JP1.3; no longer JP1.4
- net VDD_ADC: now also 4051.VDD, C1.+, JP1.1; no longer JP1.3
Other:
- note added: "Muxi v05"
- note removed: "Muxi 0.3"
Changed lines of the file:
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@@
 <?xml version="1.0" encoding="utf-8"?>
 <!DOCTYPE eagle SYSTEM "eagle.dtd">
-<eagle version="7.7.0">
+<eagle version="9.0.0">
 <drawing>
 <settings>
 <setting alwaysvectorfont="no"/>
+<setting keepoldvectorfont="yes"/>
 <setting verticaltext="up"/>
 </settings>
@@
 <layer number="113" name="IDFDebug" color="4" fill="1" visible="yes" active="yes"/>
 <layer number="116" name="Patch_BOT" color="9" fill="4" visible="yes" active="yes"/>
+<layer number="118" name="Rect_Pads" color="7" fill="1" visible="no" active="no"/>
 <layer number="121" name="_tsilk" color="7" fill="1" visible="yes" active="yes"/>
 <layer number="122" name="_bsilk" color="7" fill="1" visible="yes" active="yes"/>
@@
 <layer number="223" name="223bmp" color="24" fill="1" visible="no" active="no"/>
 <layer number="224" name="224bmp" color="25" fill="1" visible="no" active="no"/>
+<layer number="231" name="Eagle3D_PG1" color="7" fill="1" visible="no" active="no"/>
+<layer number="232" name="Eagle3D_PG2" color="7" fill="1" visible="no" active="no"/>
+<layer number="233" name="Eagle3D_PG3" color="7" fill="1" visible="no" active="no"/>
 <layer number="248" name="Housing" color="7" fill="1" visible="yes" active="yes"/>
 <layer number="249" name="Edge" color="7" fill="1" visible="yes" active="yes"/>
@@
 <parts>
 <part name="4051" library="my4051" deviceset="CD4051BE" device=""/>
-<part name="JP1" library="SparkFun-Connectors" deviceset="M08" device=""/>
 <part name="C1" library="SparkFun-Capacitors" deviceset="CAP_POL" device="PTH2"/>
 <part name="1" library="SparkFun-Connectors" deviceset="M03" device="PTH"/>
@@
 <part name="8" library="SparkFun-Connectors" deviceset="M03" device="PTH"/>
 <part name="R8" library="SparkFun-Resistors" deviceset="RESISTOR" device="AXIAL-0.3"/>
+<part name="JP1" library="SparkFun-Connectors" deviceset="M06" device="NO_SILK"/>
 </parts>
 <sheets>
 <sheet>
 <plain>
-<text x="-50.8" y="45.72" size="1.778" layer="91">Muxi 0.3</text>
+<text x="-50.8" y="45.72" size="1.778" layer="91">Muxi v05</text>
 </plain>
 <instances>
 <instance part="4051" gate="A" x="0" y="0"/>
-<instance part="JP1" gate="G$1" x="-93.98" y="30.48"/>
 <instance part="C1" gate="G$1" x="-63.5" y="33.02"/>
 <instance part="1" gate="G$1" x="-96.52" y="5.08"/>
@@
 <instance part="8" gate="G$1" x="-96.52" y="-119.38"/>
 <instance part="R8" gate="G$1" x="-63.5" y="-121.92" rot="R180"/>
+<instance part="JP1" gate="G$1" x="-93.98" y="33.02"/>
 </instances>
 <busses>
@@
 <net name="VDD_ADC" class="0">
 <segment>
-<pinref part="JP1" gate="G$1" pin="3"/>
-<wire x1="-88.9" y1="27.94" x2="-86.36" y2="27.94" width="0.1524" layer="91"/>
-<label x="-86.36" y="27.94" size="1.778" layer="95"/>
-</segment>
-<segment>
 <pinref part="1" gate="G$1" pin="1"/>
 <wire x1="-88.9" y1="2.54" x2="-86.36" y2="2.54" width="0.1524" layer="91"/>
@@
 <label x="-86.36" y="-121.92" size="1.778" layer="95"/>
 </segment>
+<segment>
+<pinref part="4051" gate="A" pin="VDD"/>
+<wire x1="-27.94" y1="7.62" x2="-30.48" y2="7.62" width="0.1524" layer="91"/>
+<label x="-40.64" y="7.62" size="1.778" layer="95"/>
+</segment>
+<segment>
+<pinref part="C1" gate="G$1" pin="+"/>
+<wire x1="-63.5" y1="35.56" x2="-63.5" y2="38.1" width="0.1524" layer="91"/>
+<label x="-63.5" y="38.1" size="1.778" layer="95"/>
+</segment>
+<segment>
+<pinref part="JP1" gate="G$1" pin="1"/>
+<wire x1="-88.9" y1="27.94" x2="-86.36" y2="27.94" width="0.1524" layer="91"/>
+<label x="-86.36" y="27.94" size="1.778" layer="95"/>
+</segment>
 </net>
 <net name="GNDA_ADC" class="0">
-<segment>
-<pinref part="JP1" gate="G$1" pin="4"/>
-<wire x1="-88.9" y1="30.48" x2="-86.36" y2="30.48" width="0.1524" layer="91"/>
-<label x="-86.36" y="30.48" size="1.778" layer="95"/>
-</segment>
 <segment>
 <pinref part="R1" gate="G$1" pin="2"/>
@@
 <wire x1="-88.9" y1="-116.84" x2="-86.36" y2="-116.84" width="0.1524" layer="91"/>
 <label x="-86.36" y="-116.84" size="1.778" layer="95"/>
+</segment>
+<segment>
+<pinref part="4051" gate="A" pin="INH"/>
+<wire x1="-27.94" y1="-10.16" x2="-30.48" y2="-10.16" width="0.1524" layer="91"/>
+<label x="-38.1" y="-10.16" size="1.778" layer="95"/>
+</segment>
+<segment>
+<pinref part="4051" gate="A" pin="VSS"/>
+<wire x1="-27.94" y1="-15.24" x2="-30.48" y2="-15.24" width="0.1524" layer="91"/>
+<label x="-38.1" y="-15.24" size="1.778" layer="95"/>
+</segment>
+<segment>
+<pinref part="4051" gate="A" pin="VEE"/>
+<wire x1="-27.94" y1="2.54" x2="-30.48" y2="2.54" width="0.1524" layer="91"/>
+<label x="-38.1" y="2.54" size="1.778" layer="95"/>
+</segment>
+<segment>
+<pinref part="C1" gate="G$1" pin="-"/>
+<wire x1="-63.5" y1="27.94" x2="-63.5" y2="25.4" width="0.1524" layer="91"/>
+<label x="-63.5" y="25.4" size="1.778" layer="95"/>
+</segment>
+<segment>
+<pinref part="JP1" gate="G$1" pin="3"/>
+<wire x1="-88.9" y1="33.02" x2="-86.36" y2="33.02" width="0.1524" layer="91"/>
+<label x="-86.36" y="33.02" size="1.778" layer="95"/>
 </segment>
 </net>
@@
 </segment>
 <segment>
-<pinref part="JP1" gate="G$1" pin="5"/>
-<wire x1="-88.9" y1="33.02" x2="-86.36" y2="33.02" width="0.1524" layer="91"/>
-<label x="-86.36" y="33.02" size="1.778" layer="95"/>
+<pinref part="JP1" gate="G$1" pin="4"/>
+<wire x1="-88.9" y1="35.56" x2="-86.36" y2="35.56" width="0.1524" layer="91"/>
+<label x="-86.36" y="35.56" size="1.778" layer="95"/>
 </segment>
 </net>
@@
 </segment>
 <segment>
-<pinref part="JP1" gate="G$1" pin="6"/>
-<wire x1="-88.9" y1="35.56" x2="-86.36" y2="35.56" width="0.1524" layer="91"/>
-<label x="-86.36" y="35.56" size="1.778" layer="95"/>
+<pinref part="JP1" gate="G$1" pin="5"/>
+<wire x1="-88.9" y1="38.1" x2="-86.36" y2="38.1" width="0.1524" layer="91"/>
+<label x="-86.36" y="38.1" size="1.778" layer="95"/>
 </segment>
 </net>
@@
 </segment>
 <segment>
-<pinref part="JP1" gate="G$1" pin="7"/>
-<wire x1="-88.9" y1="38.1" x2="-86.36" y2="38.1" width="0.1524" layer="91"/>
-<label x="-86.36" y="38.1" size="1.778" layer="95"/>
-</segment>
-</net>
-<net name="VDD_3V3" class="0">
-<segment>
-<pinref part="4051" gate="A" pin="VDD"/>
-<wire x1="-27.94" y1="7.62" x2="-30.48" y2="7.62" width="0.1524" layer="91"/>
-<label x="-40.64" y="7.62" size="1.778" layer="95"/>
-</segment>
-<segment>
-<pinref part="JP1" gate="G$1" pin="1"/>
-<wire x1="-88.9" y1="22.86" x2="-86.36" y2="22.86" width="0.1524" layer="91"/>
-<label x="-86.36" y="22.86" size="1.778" layer="95"/>
-</segment>
-<segment>
-<pinref part="C1" gate="G$1" pin="+"/>
-<wire x1="-63.5" y1="35.56" x2="-63.5" y2="38.1" width="0.1524" layer="91"/>
-<label x="-63.5" y="38.1" size="1.778" layer="95"/>
-</segment>
-</net>
-<net name="DGND" class="0">
-<segment>
-<pinref part="4051" gate="A" pin="VSS"/>
-<wire x1="-27.94" y1="-15.24" x2="-30.48" y2="-15.24" width="0.1524" layer="91"/>
-<label x="-38.1" y="-15.24" size="1.778" layer="95"/>
-</segment>
-<segment>
-<pinref part="4051" gate="A" pin="VEE"/>
-<wire x1="-27.94" y1="2.54" x2="-30.48" y2="2.54" width="0.1524" layer="91"/>
-<label x="-38.1" y="2.54" size="1.778" layer="95"/>
-</segment>
-<segment>
-<pinref part="4051" gate="A" pin="INH"/>
-<wire x1="-27.94" y1="-10.16" x2="-30.48" y2="-10.16" width="0.1524" layer="91"/>
-<label x="-38.1" y="-10.16" size="1.778" layer="95"/>
-</segment>
-<segment>
-<pinref part="JP1" gate="G$1" pin="2"/>
-<wire x1="-88.9" y1="25.4" x2="-86.36" y2="25.4" width="0.1524" layer="91"/>
-<label x="-86.36" y="25.4" size="1.778" layer="95"/>
-</segment>
-<segment>
-<pinref part="C1" gate="G$1" pin="-"/>
-<wire x1="-63.5" y1="27.94" x2="-63.5" y2="25.4" width="0.1524" layer="91"/>
-<label x="-63.5" y="25.4" size="1.778" layer="95"/>
-</segment>
-</net>
-<net name="AOUT" class="0">
-<segment>
-<pinref part="JP1" gate="G$1" pin="8"/>
+<pinref part="JP1" gate="G$1" pin="6"/>
 <wire x1="-88.9" y1="40.64" x2="-86.36" y2="40.64" width="0.1524" layer="91"/>
 <label x="-86.36" y="40.64" size="1.778" layer="95"/>
 </segment>
+</net>
+<net name="AOUT" class="0">
 <segment>
 <pinref part="4051" gate="A" pin="COM_OUT/IN"/>
@@
 <label x="30.48" y="-15.24" size="1.778" layer="95"/>
 </segment>
-</net>
+<segment>
+<pinref part="JP1" gate="G$1" pin="2"/>
+<wire x1="-88.9" y1="30.48" x2="-86.36" y2="30.48" width="0.1524" layer="91"/>
+<label x="-86.36" y="30.48" size="1.778" layer="95"/>
+</segment>
+</net>
